File: Hardware/design_bci.brd (EAGLE design)
At the start: 100 x 80 mm, 10 parts, among them IC1 AD623N

Commit message: updated
Parts:
- removed C4, C5: (no value), LinnesLab-Passives:C0603
- added B1: ARDUINO_UNO_R3_SHIELDNOLABELS, LinnesLab-Microcontrollers:UNO_R3_SHIELD_NOLABELS
- added J1: (no value), LinnesLab-Connectors:AUDIO_JACK_3.5MM_TRRS_SMD_RA
- added OP1: (no value), LinnesLab-AnalogIC:SO8
- added R5: (no value), LinnesLab-Passives:R0603
- moved C3 44.5 mm to (-22.9, 19.1)
- moved R4 44.5 mm to (-22.9, 22.9)
- moved R3 41.0 mm to (-19.1, 22.9)
- moved R2 37.9 mm to (-15.2, 22.9)
- moved C2 29.6 mm to (-19.1, 19.1)
- moved C1 26.9 mm to (-15.2, 19.1)
- moved R1 21.7 mm to (-26.7, 19.1)
Connections:
- removed net 5V: C2.1, IC1.7, R3.2
- removed net N$4 (its old number): R3.1, R4.2
- new net 3.3V: C2.1, C3.1, IC1.7, OP1.8, R4.2
- new net N$3: OP1.3, R3.2, R4.1
- new net N$6: IC1.5, OP1.1, OP1.2, OP1.5
- new net N$7: OP1.6, R1.2, R5.1
- new net N$8: OP1.7, R5.2
- net GND: now also C3.2, OP1.4, R3.1; no longer C4.2, R4.1
- net N$1: now also IC1.8, R2.2; no longer IC1.1, R1.2
- net N$2: now also IC1.1, R2.1; no longer IC1.8, R1.1
- net N$5: now also R1.1; no longer R2.1
Other:
- board size 100 x 80 mm -> 182.6 x 115.6 mm

Commit message: updated
Parts:
- moved R1 70.4 mm to (43.2, 27.9), turned to 270 degrees
- moved C2 65.4 mm to (45.7, 27.9), turned to 270 degrees
- moved IC1 65.1 mm to (41.9, 27.9)
- moved OP1 63.2 mm to (35.6, 17.8)
- moved R5 62.2 mm to (35.6, 24.1), turned to 180 degrees
- moved C1 60.4 mm to (43.2, 34.3), turned to 180 degrees
- moved R4 57.4 mm to (34.3, 17.8), turned to 90 degrees
- moved R3 56.8 mm to (36.8, 12.7), turned to 180 degrees
- moved R2 53.6 mm to (38.1, 27.9), turned to 90 degrees
- moved C3 52.2 mm to (29.2, 15.2)
- moved J1 32.4 mm to (52.1, 68.6), turned to 270 degrees
Routing:
- net 3.3V: track 0.00 -> 9.98 mm
- net GND: track 0.00 -> 6.90 mm
- net N$4: track 0.00 -> 3.15 mm
- net N$2: track 0.00 -> 2.96 mm
- net N$1: track 0.00 -> 2.96 mm

Commit message: updated
Parts:
- moved C3 10.5 mm to (39.4, 17.8), turned to 270 degrees
- moved R1 8.98 mm to (36.8, 34.3), turned to 180 degrees
- moved C2 1.27 mm to (45.7, 29.2)
- moved R5 1.27 mm to (35.6, 22.9)
- moved R3 1.27 mm to (35.6, 12.7)
Routing:
- net N$6: track 0.00 -> 39.6 mm
- net GND: track 6.90 -> 45.6 mm
- net 3.3V: track 9.98 -> 35.8 mm
- net N$7: track 0.00 -> 14.2 mm
- net N$3: track 0.00 -> 5.99 mm
- net N$5: track 0.00 -> 4.65 mm
- net N$8: track 0.00 -> 2.57 mm

Commit message: updated
Parts:
- removed B1: ARDUINO_UNO_R3_SHIELDNOLABELS, LinnesLab-Microcontrollers:UNO_R3_SHIELD_NOLABELS
- added B2: ARDUINO_UNO_R3_SHIELD_ICSP, LinnesLab-Microcontrollers:UNO_R3_SHIELD_ICSP
- moved R3 43.7 mm to (10.2, 48.3), turned to 270 degrees
- moved C3 39.5 mm to (17.8, 50.8)
- moved OP1 34.1 mm to (11.4, 41.9), turned to 180 degrees
- moved R4 31.4 mm to (17.8, 44.5), turned to 270 degrees
- moved C2 27.5 mm to (22.9, 44.5)
- moved R5 27.3 mm to (11.4, 35.6), turned to 351.8 degrees
- moved IC1 26.2 mm to (21.6, 44.5), turned to 180 degrees
- moved R1 25.4 mm to (11.4, 33.0)
- moved C1 23.0 mm to (20.3, 36.8)
- moved R2 20.8 mm to (25.4, 44.5)
Connections:
- new net N$10: IC1.2, J1.LEFT
- new net N$9: IC1.3, J1.RIGHT
- net GND: now also J1.GND, J1.GND/MIC
Routing:
- net N$6: track 39.6 -> 7.52 mm
- net 3.3V: track 35.8 -> 12.6 mm
- net GND: track 45.6 -> 25.5 mm
- net N$7: track 14.2 -> 7.64 mm
- net N$3: track 5.99 -> 11.2 mm
- net N$5: track 4.65 -> 8.77 mm
- net N$2: track 2.96 -> 5.99 mm
- net N$1: track 2.96 -> 5.68 mm
- net N$4: track 3.15 -> 5.06 mm
- net N$8: track 2.57 -> 3.96 mm
Other:
- board size 182.6 x 115.6 mm -> 53.3 x 59.7 mm

Commit message: updated
Parts:
- moved J1 15.5 mm to (39.4, 59.7)
Routing:
- net GND: track 25.5 -> 64.6 mm
- net N$9: track 0.00 -> 26.0 mm
- net N$10: track 0.00 -> 20.3 mm
- net N$6: track 7.52 -> 21.8 mm
- net 3.3V: track 12.6 -> 17.3 mm
Changed lines of the file:
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@@
 <attribute name="VALUE" x="6.985" y="43.815" size="1.27" layer="27" rot="R270"/>
 </element>
-<element name="J1" library="LinnesLab-Connectors" package="AUDIO_JACK_3.5MM_TRRS_SMD_RA" package3d_urn="urn:adsk.eagle:package:18169774/2" value="" x="52.07" y="68.58" smashed="yes" rot="R270">
-<attribute name="PROD_ID" value="CONN-10676" x="52.07" y="68.58" size="1.778" layer="27" rot="R270" display="off"/>
-<attribute name="SF_ID" value="PRT-12639" x="52.07" y="68.58" size="1.778" layer="27" rot="R270" display="off"/>
-<attribute name="VALUE" x="50.673" y="65.405" size="0.7112" layer="27" ratio="20" rot="R270"/>
+<element name="J1" library="LinnesLab-Connectors" package="AUDIO_JACK_3.5MM_TRRS_SMD_RA" package3d_urn="urn:adsk.eagle:package:18169774/2" value="" x="39.37" y="59.69" smashed="yes" rot="R270">
+<attribute name="PROD_ID" value="CONN-10676" x="39.37" y="59.69" size="1.778" layer="27" rot="R270" display="off"/>
+<attribute name="SF_ID" value="PRT-12639" x="39.37" y="59.69" size="1.778" layer="27" rot="R270" display="off"/>
+<attribute name="VALUE" x="37.973" y="56.515" size="0.7112" layer="27" ratio="20" rot="R270"/>
 </element>
 <element name="B2" library="LinnesLab-Microcontrollers" package="UNO_R3_SHIELD_ICSP" value="ARDUINO_UNO_R3_SHIELD_ICSP" x="26.67" y="30.48" smashed="yes">
@@
 <contactref element="IC1" pad="8"/>
 <contactref element="R2" pad="2"/>
-<wire x1="25.4" y1="40.64" x2="25.4" y2="42.8714" width="0.1524" layer="1"/>
+<wire x1="25.4" y1="42.8714" x2="25.4" y2="40.64" width="0.1524" layer="1"/>
 <wire x1="25.4" y1="42.8714" x2="24.7553125" y2="42.8714" width="0.1524" layer="1"/>
 <wire x1="24.7553125" y1="42.8714" x2="24.6214" y2="43.0053125" width="0.1524" layer="1"/>
@@
 <wire x1="22.2153125" y1="46.0286" x2="22.2653125" y2="46.0786" width="0.1524" layer="1"/>
 <wire x1="17.78" y1="46.0286" x2="22.2153125" y2="46.0286" width="0.1524" layer="1"/>
-<wire x1="48.82" y1="57.28" x2="55.32" y2="65.38" width="0" layer="19" extent="1-1"/>
-<wire x1="22.86" y1="43.6" x2="48.82" y2="57.28" width="0" layer="19" extent="1-1"/>
+<wire x1="24.511" y1="48.6282375" x2="25.0317625" y2="49.149" width="0.1524" layer="1"/>
+<wire x1="25.0317625" y1="49.149" x2="25.7682375" y2="49.149" width="0.1524" layer="1"/>
+<wire x1="22.86" y1="43.6" x2="24.511" y2="45.251" width="0.1524" layer="1"/>
+<wire x1="24.511" y1="45.251" x2="24.511" y2="48.6282375" width="0.1524" layer="1"/>
+<wire x1="43.18" y1="56.49" x2="42.62" y2="56.49" width="0.1524" layer="1"/>
+<wire x1="26.5272375" y1="48.39" x2="36.12" y2="48.39" width="0.1524" layer="1"/>
+<wire x1="25.7682375" y1="49.149" x2="26.5272375" y2="48.39" width="0.1524" layer="1"/>
+<wire x1="42.62" y1="56.49" x2="43.23" y2="55.88" width="0.1524" layer="1"/>
+<wire x1="43.23" y1="55.88" x2="45.72" y2="55.88" width="0.1524" layer="1"/>
+<wire x1="45.72" y1="55.88" x2="45.72" y2="48.26" width="0.1524" layer="1"/>
+<wire x1="36.25" y1="48.26" x2="36.12" y2="48.39" width="0.1524" layer="1"/>
+<wire x1="45.72" y1="48.26" x2="36.25" y2="48.26" width="0.1524" layer="1"/>
 </signal>
 <signal name="N$4">
@@
 <wire x1="10.2664" y1="40.5046875" x2="12.065" y2="42.3032875" width="0.1524" layer="1"/>
 <wire x1="12.065" y1="44.51" x2="13.335" y2="44.51" width="0.1524" layer="1"/>
-<wire x1="13.335" y1="44.51" x2="17.78" y2="40.64" width="0" layer="19" extent="1-1"/>
+<wire x1="12.8064" y1="40.5046875" x2="12.8064" y2="38.1153125" width="0.1524" layer="1"/>
+<wire x1="12.8064" y1="38.1153125" x2="12.9403125" y2="37.9814" width="0.1524" layer="1"/>
+<wire x1="12.9403125" y1="37.9814" x2="13.7296875" y2="37.9814" width="0.1524" layer="1"/>
+<wire x1="13.7296875" y1="37.9814" x2="13.8482875" y2="38.1" width="0.1524" layer="1"/>
+<wire x1="13.8482875" y1="38.1" x2="17.78" y2="38.1" width="0.1524" layer="1"/>
+<wire x1="13.335" y1="44.51" x2="13.335" y2="41.0332875" width="0.1524" layer="1"/>
+<wire x1="13.335" y1="41.0332875" x2="12.8064" y2="40.5046875" width="0.1524" layer="1"/>
+<wire x1="17.78" y1="38.1" x2="17.78" y2="40.64" width="0.1524" layer="1"/>
 </signal>
 <signal name="N$7">
@@
 <wire x1="21.16" y1="43.6" x2="22.86" y2="45.3" width="0.1524" layer="1"/>
 <wire x1="17.78" y1="43.6" x2="17.78" y2="51.65" width="0" layer="19" extent="1-1"/>
-<wire x1="22.86" y1="40.64" x2="22.86" y2="45.3" width="0" layer="19" extent="1-1"/>
+<wire x1="22.86" y1="44.45" x2="22.86" y2="45.3" width="0" layer="19" extent="1-1"/>
+<wire x1="22.1314" y1="42.9553125" x2="22.1314" y2="44.2446875" width="0.1524" layer="1"/>
+<wire x1="22.1314" y1="44.2446875" x2="22.2653125" y2="44.3786" width="0.1524" layer="1"/>
+<wire x1="22.86" y1="40.64" x2="22.86" y2="42.2267125" width="0.1524" layer="1"/>
+<wire x1="22.2653125" y1="44.3786" x2="22.7886" y2="44.3786" width="0.1524" layer="1"/>
+<wire x1="22.7886" y1="44.3786" x2="22.86" y2="44.45" width="0.1524" layer="1"/>
+<wire x1="22.86" y1="42.2267125" x2="22.1314" y2="42.9553125" width="0.1524" layer="1"/>
 </signal>
 <signal name="N$9">
 <contactref element="IC1" pad="3"/>
 <contactref element="J1" pad="RIGHT"/>
-<wire x1="55.32" y1="62.38" x2="20.32" y2="48.26" width="0" layer="19" extent="1-1"/>
+<wire x1="20.32" y1="48.26" x2="20.32" y2="50.8" width="0.1524" layer="1"/>
+<wire x1="20.32" y1="50.8" x2="22.86" y2="53.34" width="0.1524" layer="1"/>
+<wire x1="42.47" y1="53.34" x2="42.62" y2="53.49" width="0.1524" layer="1"/>
+<wire x1="22.86" y1="53.34" x2="42.47" y2="53.34" width="0.1524" layer="1"/>
 </signal>
 <signal name="N$10">
 <contactref element="IC1" pad="2"/>
 <contactref element="J1" pad="LEFT"/>
-<wire x1="22.86" y1="48.26" x2="55.32" y2="58.38" width="0" layer="19" extent="1-1"/>
+<wire x1="22.86" y1="48.26" x2="23.71170625" y2="48.26" width="0.1524" layer="1"/>
+<wire x1="23.71170625" y1="48.26" x2="24.90550625" y2="49.4538" width="0.1524" layer="1"/>
+<wire x1="38.6690625" y1="49.3978" x2="40.0709375" y2="49.3978" width="0.1524" layer="1"/>
+<wire x1="40.0709375" y1="49.3978" x2="40.1631375" y2="49.49" width="0.1524" layer="1"/>
+<wire x1="40.1631375" y1="49.49" x2="42.62" y2="49.49" width="0.1524" layer="1"/>
+<wire x1="24.90550625" y1="49.4538" x2="38.6130625" y2="49.4538" width="0.1524" layer="1"/>
+<wire x1="38.6130625" y1="49.4538" x2="38.6690625" y2="49.3978" width="0.1524" layer="1"/>
 </signal>
 </signals>

Commit message: updated
Parts:
- added C4: (no value), LinnesLab-Passives:C0603
- turned C3 to 180 degrees
Connections:
- net 3.3V: now also B2.3.3V
- net GND: now also B2.GND@0, B2.GND@2, B2.GND_ICSP
- net N$7: now also C4.1
- net N$8: now also B2.A1, C4.2
Routing:
- net GND: track 64.6 -> 145.8 mm
- net N$8: track 3.96 -> 85.2 mm
- net 3.3V: track 17.3 -> 67.7 mm
- net N$7: track 7.64 -> 14.0 mm
- net N$4: track 5.06 -> 4.16 mm

Commit message: made unnoticeable change
Routing:
- net GND: track 145.8 -> 126.1 mm
Changed lines of the file:
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@@
 <contactref element="OP1" pad="4"/>
 <contactref element="J1" pad="GND"/>
-<contactref element="J1" pad="GND/MIC"/>
 <wire x1="9.3814" y1="46.8153125" x2="9.3814" y2="48.0046875" width="0.1524" layer="1"/>
 <wire x1="9.3814" y1="48.0046875" x2="9.5153125" y2="48.1386" width="0.1524" layer="1"/>
@@
 <wire x1="22.86" y1="43.6" x2="24.511" y2="45.251" width="0.1524" layer="1"/>
 <wire x1="24.511" y1="45.251" x2="24.511" y2="48.6282375" width="0.1524" layer="1"/>
-<wire x1="26.5272375" y1="48.39" x2="36.12" y2="48.39" width="0.1524" layer="1"/>
 <wire x1="25.7682375" y1="49.149" x2="26.5272375" y2="48.39" width="0.1524" layer="1"/>
 <wire x1="42.62" y1="56.49" x2="43.23" y2="55.88" width="0.1524" layer="1"/>
 <wire x1="43.23" y1="55.88" x2="45.72" y2="55.88" width="0.1524" layer="1"/>
 <wire x1="45.72" y1="55.88" x2="45.72" y2="48.26" width="0.1524" layer="1"/>
-<wire x1="36.25" y1="48.26" x2="36.12" y2="48.39" width="0.1524" layer="1"/>
 <wire x1="45.72" y1="48.26" x2="36.25" y2="48.26" width="0.1524" layer="1"/>
 <contactref element="B2" pad="GND@2"/>
@@
 <wire x1="27.9900125" y1="57.29000625" x2="28.88221875" y2="56.3978" width="0.1524" layer="1"/>
 <wire x1="28.88221875" y1="56.3978" x2="40.0709375" y2="56.3978" width="0.1524" layer="1"/>
-<wire x1="36.12" y1="48.39" x2="43.18" y2="41.33" width="0.1524" layer="1"/>
 <wire x1="43.18" y1="41.33" x2="43.18" y2="31.75" width="0.1524" layer="1"/>
 <wire x1="43.18" y1="31.75" x2="50.8" y2="31.75" width="0.1524" layer="1"/>
@@
 <wire x1="42.01" y1="55.88" x2="41.91" y2="55.88" width="0.1524" layer="1"/>
 <wire x1="41.91" y1="55.88" x2="41.91" y2="56.49" width="0.1524" layer="1"/>
+<contactref element="J1" pad="GND/MIC"/>
+<wire x1="36.12" y1="48.39" x2="36.25" y2="48.26" width="0" layer="19" extent="1-1"/>
+<wire x1="26.5272375" y1="48.39" x2="27.9900125" y2="57.29000625" width="0" layer="19" extent="1-1"/>
+<wire x1="43.18" y1="41.33" x2="36.25" y2="48.26" width="0" layer="19" extent="1-1"/>
 </signal>
 <signal name="N$4">

Commit message: updated
Routing:
- net GND: track 126.1 -> 199.1 mm
- added copper zone on layer 1, net 3.3V
- added copper zone on layer 16, net GND
Changed lines of the file:
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@@
 <wire x1="22.86" y1="43.6" x2="24.511" y2="45.251" width="0.1524" layer="1"/>
 <wire x1="24.511" y1="45.251" x2="24.511" y2="48.6282375" width="0.1524" layer="1"/>
-<wire x1="25.7682375" y1="49.149" x2="26.5272375" y2="48.39" width="0.1524" layer="1"/>
+<wire x1="26.5272375" y1="48.39" x2="25.7682375" y2="49.149" width="0.1524" layer="1"/>
 <wire x1="42.62" y1="56.49" x2="43.23" y2="55.88" width="0.1524" layer="1"/>
 <wire x1="43.23" y1="55.88" x2="45.72" y2="55.88" width="0.1524" layer="1"/>
-<wire x1="45.72" y1="55.88" x2="45.72" y2="48.26" width="0.1524" layer="1"/>
-<wire x1="45.72" y1="48.26" x2="36.25" y2="48.26" width="0.1524" layer="1"/>
+<wire x1="45.72" y1="48.26" x2="45.72" y2="55.88" width="0.1524" layer="1"/>
 <contactref element="B2" pad="GND@2"/>
 <contactref element="B2" pad="GND_ICSP"/>
@@
 <wire x1="41.91" y1="55.88" x2="41.91" y2="56.49" width="0.1524" layer="1"/>
 <contactref element="J1" pad="GND/MIC"/>
-<wire x1="36.12" y1="48.39" x2="36.25" y2="48.26" width="0" layer="19" extent="1-1"/>
-<wire x1="26.5272375" y1="48.39" x2="27.9900125" y2="57.29000625" width="0" layer="19" extent="1-1"/>
-<wire x1="43.18" y1="41.33" x2="36.25" y2="48.26" width="0" layer="19" extent="1-1"/>
+<wire x1="43.9752125" y1="54.344" x2="44.124" y2="54.1952125" width="0.2032" layer="1"/>
+<wire x1="44.124" y1="54.1952125" x2="44.124" y2="52.7847875" width="0.2032" layer="1"/>
+<wire x1="44.124" y1="52.7847875" x2="43.9752125" y2="52.636" width="0.2032" layer="1"/>
+<wire x1="43.9752125" y1="52.636" x2="41.2647875" y2="52.636" width="0.2032" layer="1"/>
+<wire x1="21.9456" y1="48.6387625" x2="21.9456" y2="47.8812375" width="0.2032" layer="1"/>
+<wire x1="25.0212375" y1="39.7256" x2="25.7787625" y2="39.7256" width="0.2032" layer="1"/>
+<wire x1="27.9900125" y1="57.29000625" x2="30.93601875" y2="54.344" width="0.2032" layer="1"/>
+<wire x1="41.2647875" y1="52.636" x2="41.0931875" y2="52.8076" width="0.2032" layer="1"/>
+<wire x1="30.93601875" y1="54.344" x2="43.9752125" y2="54.344" width="0.2032" layer="1"/>
+<wire x1="24.2912" y1="40.4556375" x2="25.0212375" y2="39.7256" width="0.2032" layer="1"/>
+<wire x1="41.0931875" y1="52.8076" x2="26.1144375" y2="52.8076" width="0.2032" layer="1"/>
+<wire x1="26.1144375" y1="52.8076" x2="21.9456" y2="48.6387625" width="0.2032" layer="1"/>
+<wire x1="24.2912" y1="45.5356375" x2="24.2912" y2="40.4556375" width="0.2032" layer="1"/>
+<wire x1="21.9456" y1="47.8812375" x2="24.2912" y2="45.5356375" width="0.2032" layer="1"/>
+<wire x1="26.5088" y1="48.3715625" x2="26.5272375" y2="48.39" width="0.2032" layer="1"/>
+<wire x1="25.7787625" y1="39.7256" x2="26.5088" y2="40.4556375" width="0.2032" layer="1"/>
+<wire x1="26.5088" y1="40.4556375" x2="26.5088" y2="48.3715625" width="0.2032" layer="1"/>
+<wire x1="36.12" y1="48.39" x2="43.18" y2="41.33" width="0.2032" layer="1"/>
+<polygon width="0.2032" layer="16">
+<vertex x="0" y="59.69"/>
+<vertex x="52.07" y="59.69"/>
+<vertex x="52.07" y="0"/>
+<vertex x="0" y="0"/>
+</polygon>
+<wire x1="36.12" y1="48.39" x2="45.72" y2="48.39" width="0.2032" layer="1"/>
+<wire x1="45.72" y1="48.39" x2="45.72" y2="48.26" width="0.2032" layer="1"/>
 </signal>
 <signal name="N$4">
@@
 <wire x1="19.05" y1="49.53" x2="19.05" y2="50.38" width="0.1524" layer="1"/>
 <wire x1="19.05" y1="50.38" x2="18.63" y2="50.8" width="0.1524" layer="1"/>
+<polygon width="0.2032" layer="1">
+<vertex x="0" y="59.69"/>
+<vertex x="53.34" y="59.69"/>
+<vertex x="53.34" y="0"/>
+<vertex x="0" y="0"/>
+</polygon>
 </signal>
 <signal name="N$9">
