File: Hardware/design_bci.brd (EAGLE design)
At the start: 53.3 x 59.7 mm, 13 parts, among them IC1 AD623N

Commit message: orlando made changes and ordered boards
Parts:
- moved C4 32.9 mm to (36.1, 19.0), turned to 90 degrees
- moved C3 30.2 mm to (29.7, 23.1)
- moved OP1 28.0 mm to (27.7, 19.1), turned to 270 degrees
- moved R5 27.7 mm to (33.6, 18.9), turned to 90 degrees
- moved R2 27.5 mm to (18.9, 17.7)
- moved R4 27.0 mm to (35.8, 24.3)
- moved C2 19.2 mm to (35.9, 30.4)
- moved R3 19.0 mm to (27.8, 41.2), turned to 0 degrees
- moved R1 18.3 mm to (21.3, 17.6), turned to 270 degrees
- moved C1 15.4 mm to (35.4, 33.9), turned to 0 degrees
- moved IC1 13.3 mm to (27.7, 32.6), turned to 270 degrees
- renumbered B2 to B1
Connections:
- net 3.3V: now also C1.1, R1.2; no longer C2.1, R4.2
- net GND: now also B1.GND@1, C1.2, R2.1; no longer C2.2, R3.1
- net N$1: now also R3.2; no longer R2.2
- net N$2: now also R3.1; no longer R2.1
- net N$3: now also R1.1, R2.2; no longer R3.2, R4.1
- net N$4: now also C2.1; no longer C1.1
- net N$5: now also C2.2, R4.1; no longer C1.2, R1.1
- net N$7: now also R4.2; no longer R1.2
Routing:
- net GND: track 199.1 -> 9.98 mm, vias 0 -> 6
- net 3.3V: track 67.7 -> 0.00 mm
- net N$8: track 85.2 -> 42.3 mm
- net N$10: track 20.3 -> 35.5 mm
- net N$9: track 26.0 -> 39.3 mm
- net N$3: track 11.7 -> 6.20 mm
- net N$7: track 14.0 -> 18.9 mm
- net N$5: track 8.77 -> 4.48 mm
- net N$6: track 21.8 -> 18.0 mm
