File: Hardware/design_bci.sch (EAGLE design)
At the start: 11 parts, among them IC1 AD623N

Commit message: updated
Parts:
- removed OP2: (no value), LinnesLab-AnalogIC:OP-DUALR
- added B1: ARDUINO_UNO_R3_SHIELDNOLABELS, LinnesLab-Microcontrollers:ARDUINO_UNO_R3_SHIELDNOLABELS
- added J1: (no value), LinnesLab-Connectors:AUDIO_JACK_TRRSSMD_RA
- OP1: device LinnesLab-AnalogIC:OP-DUALR -> LinnesLab-AnalogIC:OP-DUALMCP6002R
Connections:
- removed net 5V: C2.1, C3.1, IC1.+V, R4.2
- new net 3.3V: C2.1, C3.1, IC1.+V, OP1P.V+, R4.2
- new net N$6: IC1.REF, OP1A.-IN, OP1A.OUT, OP1B.+IN
- new net N$7: OP1B.-IN, R1.2, R5.1
- new net N$8: OP1B.OUT, R5.2
- net GND: now also OP1P.V-
- net N$3: now also OP1A.+IN
Other:
- moved on the sheet: OP1A, OP1B, OP1P

Commit message: updated
Parts:
- removed B1: ARDUINO_UNO_R3_SHIELDNOLABELS, LinnesLab-Microcontrollers:ARDUINO_UNO_R3_SHIELDNOLABELS
- added B2: ARDUINO_UNO_R3_SHIELD_ICSP, LinnesLab-Microcontrollers:ARDUINO_UNO_R3_SHIELD_ICSP
Connections:
- new net N$10: IC1.-, J1.TIP
- new net N$9: IC1.+, J1.RING1
- net GND: now also J1.RING2, J1.SLEEVE
Other:
- moved on the sheet: J1
Changed lines of the file:
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@@
 <part name="SUPPLY2" library="LinnesLab-Symbols" deviceset="3.3V" device=""/>
 <part name="SUPPLY3" library="LinnesLab-Symbols" deviceset="3.3V" device=""/>
-<part name="B1" library="LinnesLab-Microcontrollers" deviceset="ARDUINO_UNO_R3_SHIELD" device="NOLABELS"/>
 <part name="J1" library="LinnesLab-Connectors" deviceset="AUDIO_JACK_TRRS" device="SMD_RA" package3d_urn="urn:adsk.eagle:package:18169774/2"/>
+<part name="B2" library="LinnesLab-Microcontrollers" deviceset="ARDUINO_UNO_R3_SHIELD_ICSP" device=""/>
+<part name="GND6" library="LinnesLab-Symbols" deviceset="GND" device=""/>
+<part name="GND7" library="LinnesLab-Symbols" deviceset="GND" device=""/>
 </parts>
 <sheets>
@@
 <attribute name="VALUE" x="76.2" y="61.214" size="1.778" layer="96" align="bottom-center"/>
 </instance>
-<instance part="B1" gate="G$1" x="99.06" y="20.32" smashed="yes">
-<attribute name="NAME" x="89.408" y="40.894" size="1.778" layer="95" font="vector"/>
-<attribute name="VALUE" x="90.17" y="-5.334" size="1.778" layer="96" font="vector" align="top-left"/>
-</instance>
-<instance part="J1" gate="G$1" x="53.34" y="5.08" smashed="yes">
-<attribute name="NAME" x="48.26" y="10.668" size="1.778" layer="95"/>
-<attribute name="VALUE" x="48.26" y="-2.54" size="1.778" layer="96"/>
+<instance part="J1" gate="G$1" x="-7.62" y="88.9" smashed="yes">
+<attribute name="NAME" x="-12.7" y="94.488" size="1.778" layer="95"/>
+<attribute name="VALUE" x="-12.7" y="81.28" size="1.778" layer="96"/>
+</instance>
+<instance part="B2" gate="G$1" x="99.06" y="35.56" smashed="yes">
+<attribute name="NAME" x="89.408" y="66.802" size="1.778" layer="95" font="vector"/>
+<attribute name="VALUE" x="88.9" y="4.826" size="1.778" layer="96" font="vector" align="top-left"/>
+</instance>
+<instance part="GND6" gate="G$1" x="-2.54" y="76.2" smashed="yes">
+<attribute name="VALUE" x="-2.54" y="75.946" size="1.778" layer="96" align="top-center"/>
+</instance>
+<instance part="GND7" gate="G$1" x="2.54" y="78.74" smashed="yes">
+<attribute name="VALUE" x="2.54" y="78.486" size="1.778" layer="96" align="top-center"/>
 </instance>
 </instances>
@@
 <pinref part="OP1" gate="P" pin="V-"/>
 <wire x1="76.2" y1="38.1" x2="76.2" y2="40.64" width="0.1524" layer="91"/>
+</segment>
+<segment>
+<pinref part="J1" gate="G$1" pin="RING2"/>
+<wire x1="-2.54" y1="83.82" x2="-2.54" y2="78.74" width="0.1524" layer="91"/>
+<pinref part="GND6" gate="G$1" pin="GND"/>
+</segment>
+<segment>
+<pinref part="J1" gate="G$1" pin="SLEEVE"/>
+<wire x1="-2.54" y1="93.98" x2="2.54" y2="93.98" width="0.1524" layer="91"/>
+<wire x1="2.54" y1="93.98" x2="2.54" y2="81.28" width="0.1524" layer="91"/>
+<pinref part="GND7" gate="G$1" pin="GND"/>
+<wire x1="2.54" y1="81.28" x2="2.54" y2="78.74" width="0.1524" layer="91"/>
+<junction x="2.54" y="81.28"/>
 </segment>
 </net>
@@
 </segment>
 </net>
+<net name="N$9" class="0">
+<segment>
+<pinref part="IC1" gate="G$1" pin="+"/>
+<wire x1="12.7" y1="96.52" x2="7.62" y2="96.52" width="0.1524" layer="91"/>
+<wire x1="7.62" y1="96.52" x2="7.62" y2="91.44" width="0.1524" layer="91"/>
+<pinref part="J1" gate="G$1" pin="RING1"/>
+<wire x1="7.62" y1="91.44" x2="-2.54" y2="91.44" width="0.1524" layer="91"/>
+</segment>
+</net>
+<net name="N$10" class="0">
+<segment>
+<pinref part="IC1" gate="G$1" pin="-"/>
+<wire x1="12.7" y1="76.2" x2="7.62" y2="76.2" width="0.1524" layer="91"/>
+<wire x1="7.62" y1="76.2" x2="7.62" y2="86.36" width="0.1524" layer="91"/>
+<pinref part="J1" gate="G$1" pin="TIP"/>
+<wire x1="7.62" y1="86.36" x2="-2.54" y2="86.36" width="0.1524" layer="91"/>
+</segment>
+</net>

Commit message: updated
Parts:
- added C4: (no value), LinnesLab-Passives:CAPACITOR0603
Connections:
- net 3.3V: now also B2.3.3V
- net GND: now also B2.GND, B2.GND@0, B2.GND@2
- net N$7: now also C4.1
- net N$8: now also B2.A1, C4.2
Other:
- moved on the sheet: B2
Changed lines of the file:
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@@
 <part name="GND6" library="LinnesLab-Symbols" deviceset="GND" device=""/>
 <part name="GND7" library="LinnesLab-Symbols" deviceset="GND" device=""/>
+<part name="SUPPLY4" library="LinnesLab-Symbols" deviceset="3.3V" device=""/>
+<part name="C4" library="LinnesLab-Passives" deviceset="CAPACITOR" device="0603" package3d_urn="urn:adsk.eagle:package:15661989/2"/>
+<part name="GND8" library="LinnesLab-Symbols" deviceset="GND" device=""/>
 </parts>
 <sheets>
@@
 <attribute name="VALUE" x="-12.7" y="81.28" size="1.778" layer="96"/>
 </instance>
-<instance part="B2" gate="G$1" x="99.06" y="35.56" smashed="yes">
-<attribute name="NAME" x="89.408" y="66.802" size="1.778" layer="95" font="vector"/>
-<attribute name="VALUE" x="88.9" y="4.826" size="1.778" layer="96" font="vector" align="top-left"/>
+<instance part="B2" gate="G$1" x="121.92" y="71.12" smashed="yes">
+<attribute name="NAME" x="112.268" y="102.362" size="1.778" layer="95" font="vector"/>
+<attribute name="VALUE" x="111.76" y="40.386" size="1.778" layer="96" font="vector" align="top-left"/>
 </instance>
 <instance part="GND6" gate="G$1" x="-2.54" y="76.2" smashed="yes">
@@
 <instance part="GND7" gate="G$1" x="2.54" y="78.74" smashed="yes">
 <attribute name="VALUE" x="2.54" y="78.486" size="1.778" layer="96" align="top-center"/>
+</instance>
+<instance part="SUPPLY4" gate="G$1" x="106.68" y="71.12" smashed="yes">
+<attribute name="VALUE" x="106.68" y="73.914" size="1.778" layer="96" align="bottom-center"/>
+</instance>
+<instance part="C4" gate="G$1" x="88.9" y="124.46" smashed="yes" rot="R90">
+<attribute name="NAME" x="85.979" y="125.984" size="1.778" layer="95" rot="R180"/>
+<attribute name="VALUE" x="91.059" y="125.984" size="1.778" layer="96" rot="R90"/>
+</instance>
+<instance part="GND8" gate="G$1" x="106.68" y="38.1" smashed="yes">
+<attribute name="VALUE" x="106.68" y="37.846" size="1.778" layer="96" align="top-center"/>
 </instance>
 </instances>
@@
 <wire x1="2.54" y1="81.28" x2="2.54" y2="78.74" width="0.1524" layer="91"/>
 <junction x="2.54" y="81.28"/>
+</segment>
+<segment>
+<pinref part="B2" gate="G$1" pin="GND@2"/>
+<wire x1="109.22" y1="66.04" x2="106.68" y2="66.04" width="0.1524" layer="91"/>
+<pinref part="GND8" gate="G$1" pin="GND"/>
+<wire x1="106.68" y1="66.04" x2="106.68" y2="60.96" width="0.1524" layer="91"/>
+<pinref part="B2" gate="G$1" pin="GND"/>
+<wire x1="106.68" y1="60.96" x2="106.68" y2="43.18" width="0.1524" layer="91"/>
+<wire x1="106.68" y1="43.18" x2="106.68" y2="40.64" width="0.1524" layer="91"/>
+<wire x1="109.22" y1="43.18" x2="106.68" y2="43.18" width="0.1524" layer="91"/>
+<junction x="106.68" y="43.18"/>
+<pinref part="B2" gate="G$1" pin="GND@0"/>
+<wire x1="109.22" y1="60.96" x2="106.68" y2="60.96" width="0.1524" layer="91"/>
+<junction x="106.68" y="60.96"/>
 </segment>
 </net>
@@
 <wire x1="73.66" y1="114.3" x2="88.9" y2="114.3" width="0.1524" layer="91"/>
 <pinref part="OP1" gate="B" pin="-IN"/>
+<wire x1="73.66" y1="114.3" x2="73.66" y2="124.46" width="0.1524" layer="91"/>
+<junction x="73.66" y="114.3"/>
+<pinref part="C4" gate="G$1" pin="1"/>
+<wire x1="73.66" y1="124.46" x2="83.82" y2="124.46" width="0.1524" layer="91"/>
 </segment>
 </net>
@@
 <wire x1="104.14" y1="96.52" x2="101.6" y2="96.52" width="0.1524" layer="91"/>
 <pinref part="OP1" gate="B" pin="OUT"/>
+<pinref part="C4" gate="G$1" pin="2"/>
+<wire x1="91.44" y1="124.46" x2="104.14" y2="124.46" width="0.1524" layer="91"/>
+<wire x1="104.14" y1="124.46" x2="104.14" y2="114.3" width="0.1524" layer="91"/>
+<junction x="104.14" y="114.3"/>
+<pinref part="B2" gate="G$1" pin="A1"/>
+<wire x1="109.22" y1="96.52" x2="104.14" y2="96.52" width="0.1524" layer="91"/>
+<junction x="104.14" y="96.52"/>
 </segment>
 </net>
@@
 <wire x1="63.5" y1="58.42" x2="63.5" y2="55.88" width="0.1524" layer="91"/>
 </segment>
-</net>
+<segment>
+<pinref part="B2" gate="G$1" pin="3.3V"/>
+<pinref part="SUPPLY4" gate="G$1" pin="3.3V"/>
+<wire x1="109.22" y1="71.12" x2="106.68" y2="71.12" width="0.1524" layer="91"/>
+</segment>
+</net>

Commit message: made unnoticeable change
Changed lines of the file:
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@@
-</segment>
-<segment>
-<pinref part="J1" gate="G$1" pin="SLEEVE"/>
-<wire x1="-2.54" y1="93.98" x2="2.54" y2="93.98" width="0.1524" layer="91"/>
-<wire x1="2.54" y1="93.98" x2="2.54" y2="81.28" width="0.1524" layer="91"/>
-<pinref part="GND7" gate="G$1" pin="GND"/>
-<wire x1="2.54" y1="81.28" x2="2.54" y2="78.74" width="0.1524" layer="91"/>
-<junction x="2.54" y="81.28"/>
 </segment>
 <segment>
@@
 <junction x="106.68" y="60.96"/>
 </segment>
+<segment>
+<pinref part="J1" gate="G$1" pin="SLEEVE"/>
+<wire x1="-2.54" y1="93.98" x2="2.54" y2="93.98" width="0.1524" layer="91"/>
+<pinref part="GND7" gate="G$1" pin="GND"/>
+<wire x1="2.54" y1="93.98" x2="2.54" y2="81.28" width="0.1524" layer="91"/>
+</segment>
 </net>

Commit message: orlando made changes and ordered boards
Parts:
- renumbered B2 to B1
Connections:
- net 3.3V: now also C1.1, R1.2; no longer C2.1, R4.2
- net GND: now also B1.GND@1, C1.2, R2.1; no longer C2.2, R3.1
- net N$1: now also R3.2; no longer R2.2
- net N$2: now also R3.1; no longer R2.1
- net N$3: now also R1.1, R2.2; no longer R3.2, R4.1
- net N$4: now also C2.1; no longer C1.1
- net N$5: now also C2.2, R4.1; no longer C1.2, R1.1
- net N$7: now also R4.2; no longer R1.2
Other:
- moved on the sheet: C1, C2, R1, R2, R3, R4
